File: KiCad Files Onboard Pico/MCU.kicad_sch (KiCad schematic)
At the start: 38 parts, among them J201 GT-USB-7051A, J203 Button, U201 TPS63001DRCR, U202 RP2040, Y201 3225_4P 12MHz

Commit message: small corrections
Parts:
- R201, R202: value 5.1K 0402 -> 5K1 0402
Changed lines of the file:
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@@
 			)
 		)
-		(property "Value" "5.1K 0402"
+		(property "Value" "5K1 0402"
 			(at 41.91 38.1 90)
 			(effects
@@
 			)
 		)
-		(property "Value" "5.1K 0402"
+		(property "Value" "5K1 0402"
 			(at 41.91 40.64 90)
 			(effects
